Commit message: make prbt compatible

File: docs/application_scan_and_plan/static/snp_prbt.urdf (robot description, URDF)
Before this commit: robot snp_psir_description, 22 links, 21 joints
Links:
- link acf_111_04_and_grinder: geometry collision cylinder length=0.04 radius=0.012; collision cylinder length=0.08 radius=0.02
- link ensenso: geometry collision box size=0.18 0.05 0.055; visual mesh filename=package://snp_prbt_description/meshes/ensenso_n35.STL
- link tool_fixture: geometry collision mesh filename=package://snp_prbt_description/meshes/tool_fixture.STL; visual mesh filename=package://snp_prbt_description/meshes/tool_fixture.STL
