Commit message: new manipulation animation

File: docs/manipulator_ur5/static/ur5_with_cam.urdf (robot description, URDF)
Before this commit: robot ur5, 11 links, 10 joints
Links:
- added link camera; visual mesh filename=package://openni_description/mesh/kinect.dae scale=2 2 2
Joints:
- added joint camera_joint: type fixed, parent tool0, child camera, origin xyz=0 0 0.05 rpy=0.0 0 0.0
